Commit message: tweeks

File: src/bringup/urdf/robot.urdf.xacro (robot description, xacro)
@@ -42,5 +42,5 @@
   </joint>
   <joint name="lidar0_joint" type="fixed">
-    <origin xyz="0.271705 0.360295 0.0" rpy="0.0 0.0 0.0" />
+    <origin xyz="0.271705 0.38160499999999997 0.0" rpy="${radians(180)} 0.0 ${radians(93)}" />
     <parent link="base_link" />
     <child link="lidar0_link" />
@@ -48,5 +48,5 @@
   </joint>
   <joint name="lidar1_joint" type="fixed">
-    <origin xyz="0.271705 0.271705 0.0" rpy="0.0 0.0 0.0" />
+    <origin xyz="0.271705 0.271705 0.0" rpy="${radians(180)} 0.0 ${radians(180)}" />
     <parent link="base_link" />
     <child link="lidar1_link" />
@@ -54,5 +54,5 @@
   </joint>
   <joint name="lidar2_joint" type="fixed">
-    <origin xyz="-0.271705 -0.271705 0.0" rpy="0.0 0.0 0.0" />
+    <origin xyz="-0.271705 -0.271705 0.0" rpy="${radians(180)} 0.0 ${radians(-90)}" />
     <parent link="base_link" />
     <child link="lidar2_link" />

Commit message: adopt the latest machine design

File: src/bringup/urdf/robot.urdf.xacro (robot description, xacro)
@@ -28,5 +28,5 @@
     </visual>
   </link>
-  <link name="lidar2_link">
+  <!-- <link name="lidar2_link">
     <visual>
       <geometry>
@@ -34,5 +34,5 @@
       </geometry>
     </visual>
-  </link>
+  </link> -->
   <joint name="base_joint" type="fixed">
     <origin xyz="0.0 0.0 0.05" rpy="0.0 0.0 0.0" />
@@ -42,5 +42,5 @@
   </joint>
   <joint name="lidar0_joint" type="fixed">
-    <origin xyz="0.271705 0.38160499999999997 0.0" rpy="${radians(180)} 0.0 ${radians(93)}" />
+    <origin xyz="0.0 -0.4 0.0" rpy="${radians(180)} 0.0 ${radians(-90)}" />
     <parent link="base_link" />
     <child link="lidar0_link" />
@@ -48,14 +48,14 @@
   </joint>
   <joint name="lidar1_joint" type="fixed">
-    <origin xyz="0.271705 0.271705 0.0" rpy="${radians(180)} 0.0 ${radians(180)}" />
+    <origin xyz="0.0 0.4 0.0" rpy="${radians(180)} 0.0 ${radians(180)}" />
     <parent link="base_link" />
     <child link="lidar1_link" />
     <axis xyz="0.0 0.0 0.0" />
   </joint>
-  <joint name="lidar2_joint" type="fixed">
+  <!-- <joint name="lidar2_joint" type="fixed">
     <origin xyz="-0.271705 -0.271705 0.0" rpy="${radians(180)} 0.0 ${radians(-90)}" />
     <parent link="base_link" />
     <child link="lidar2_link" />
     <axis xyz="0.0 0.0 0.0" />
-  </joint>
+  </joint> -->
 </robot>

Commit message: fix urdf

File: src/bringup/urdf/robot.urdf.xacro (robot description, xacro)
@@ -42,5 +42,5 @@
   </joint>
   <joint name="lidar0_joint" type="fixed">
-    <origin xyz="0.0 -0.4 0.0" rpy="${radians(180)} 0.0 ${radians(-90)}" />
+    <origin xyz="0.0 -0.4 0.0" rpy="${radians(180)} 0.0 ${radians(0)}" />
     <parent link="base_link" />
     <child link="lidar0_link" />

Commit message: many changes

File: src/bringup/urdf/robot.urdf.xacro (robot description, xacro)
@@ -42,5 +42,5 @@
   </joint>
   <joint name="lidar0_joint" type="fixed">
-    <origin xyz="0.0 -0.4 0.0" rpy="${radians(180)} 0.0 ${radians(0)}" />
+    <origin xyz="-0.175 -0.3868 0.0" rpy="${radians(180)} 0.0 ${radians(0)}" />
     <parent link="base_link" />
     <child link="lidar0_link" />
@@ -48,5 +48,5 @@
   </joint>
   <joint name="lidar1_joint" type="fixed">
-    <origin xyz="0.0 0.4 0.0" rpy="${radians(180)} 0.0 ${radians(180)}" />
+    <origin xyz="-0.175 0.3868 0.0" rpy="${radians(180)} 0.0 ${radians(180)}" />
     <parent link="base_link" />
     <child link="lidar1_link" />

Commit message: wall tracking

File: src/bringup/urdf/robot.urdf.xacro (robot description, xacro)
@@ -48,5 +48,5 @@
   </joint>
   <joint name="lidar1_joint" type="fixed">
-    <origin xyz="-0.175 0.3868 0.0" rpy="${radians(180)} 0.0 ${radians(180)}" />
+    <origin xyz="-0.175 -0.220 0.0" rpy="0.0 0.0 ${radians(0)}" />
     <parent link="base_link" />
     <child link="lidar1_link" />

Commit message: adjust lidar pose

File: src/bringup/urdf/robot.urdf.xacro (robot description, xacro)
@@ -7,5 +7,4 @@
       <geometry>
         <box size="0.54341 0.54341 0.5"/>
-        <!-- <mesh filename="package://nhka_description/models/nhka_body.stl" /> -->
       </geometry>
       <material name="gray">
@@ -28,11 +27,4 @@
     </visual>
   </link>
-  <!-- <link name="lidar2_link">
-    <visual>
-      <geometry>
-        <box size="0.05 0.05 0.05"/>
-      </geometry>
-    </visual>
-  </link> -->
   <joint name="base_joint" type="fixed">
     <origin xyz="0.0 0.0 0.05" rpy="0.0 0.0 0.0" />
@@ -42,5 +34,5 @@
   </joint>
   <joint name="lidar0_joint" type="fixed">
-    <origin xyz="-0.175 -0.3868 0.0" rpy="${radians(180)} 0.0 ${radians(0)}" />
+    <origin xyz="-0.098 -0.3797 0.0" rpy="${radians(180)} 0.0 ${radians(0)}" />
     <parent link="base_link" />
     <child link="lidar0_link" />
@@ -48,14 +40,8 @@
   </joint>
   <joint name="lidar1_joint" type="fixed">
-    <origin xyz="-0.175 -0.220 0.0" rpy="0.0 0.0 ${radians(0)}" />
+    <origin xyz="0.3645 -0.220 0.0" rpy="0.0 0.0 ${radians(0)}" />
     <parent link="base_link" />
     <child link="lidar1_link" />
     <axis xyz="0.0 0.0 0.0" />
   </joint>
-  <!-- <joint name="lidar2_joint" type="fixed">
-    <origin xyz="-0.271705 -0.271705 0.0" rpy="${radians(180)} 0.0 ${radians(-90)}" />
-    <parent link="base_link" />
-    <child link="lidar2_link" />
-    <axis xyz="0.0 0.0 0.0" />
-  </joint> -->
 </robot>

Commit message: fix urdf

File: src/bringup/urdf/robot.urdf.xacro (robot description, xacro)
@@ -34,5 +34,5 @@
   </joint>
   <joint name="lidar0_joint" type="fixed">
-    <origin xyz="-0.098 -0.3797 0.0" rpy="${radians(180)} 0.0 ${radians(0)}" />
+    <origin xyz="-0.098 -0.3797 0.0" rpy="${radians(180)} 0.0 ${radians(-90)}" />
     <parent link="base_link" />
     <child link="lidar0_link" />

Commit message: change lidar pose

File: src/bringup/urdf/robot.urdf.xacro (robot description, xacro)
@@ -34,5 +34,5 @@
   </joint>
   <joint name="lidar0_joint" type="fixed">
-    <origin xyz="-0.098 -0.3797 0.0" rpy="${radians(180)} 0.0 ${radians(-90)}" />
+    <origin xyz="-0.098 -0.3797 0.0" rpy="${radians(180)} 0.0 ${radians(90)}" />
     <parent link="base_link" />
     <child link="lidar0_link" />
